File: pcb/hotswap/cornelius.kicad_sch (KiCad schematic)
At the start: 116 parts, among them J1 AVR-ISP-6, SW1 SW_Push, U1 ATmega32U4-MU, U2 PRTR5V0U2X, Y1 16MHz

Commit message: Add hotswap pcb
Parts:
- removed MX1, MX10, MX11, MX12, MX13, MX14, MX15, MX16, MX17, MX18, MX19, MX2, MX20, MX21, MX22, MX23, MX24, MX25, MX26, MX27, MX28, MX29, MX3, MX30, MX31, MX32, MX33, MX34, MX35, MX36, MX37, MX38, MX39, MX4, MX40, MX41, MX42, MX43, MX44, MX45, MX46, MX47, MX48, MX5, MX6, MX7, MX8, MX9: MX-NoLED, MX_Only:MXOnly-1U-Hotswap, symbol cornelius-rescue:MX-NoLED-MX_Alps_Hybrid
- removed U1: ATmega32U4-MU, Housings_DFN_QFN:QFN-44-1EP_7x7mm_Pitch0.5mm, symbol cornelius-rescue:ATmega32U4-MU-MCU_Microchip_ATmega-Orbit-rescue-corne-plus-res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
- removed U2: PRTR5V0U2X, locallib:SOT143B, symbol cornelius-rescue:PRTR5V0U2X-ai03-locallib
- removed USB1: HRO-TYPE-C-31-M-12, Type-C:HRO-TYPE-C-31-M-12-Assembly, symbol cornelius-rescue:HRO-TYPE-C-31-M-12-Type-C
- added MX1, MX10, MX11, MX12, MX13, MX14, MX15, MX16, MX17, MX18, MX19, MX2, MX20, MX21, MX22, MX23, MX24, MX25, MX26, MX27, MX28, MX29, MX3, MX30, MX31, MX32, MX33, MX34, MX35, MX36, MX37, MX38, MX39, MX4, MX40, MX41, MX42, MX43, MX44, MX45, MX46, MX47, MX48, MX5, MX6, MX7, MX8, MX9: SW_Push, kbd:keyswitch_cherrymx_hotswap_1u, symbol Switch:SW_Push
- added U1: ATmega32U4-M, Package_DFN_QFN:QFN-44-1EP_7x7mm_P0.5mm_EP5.2x5.2mm, symbol MCU_Microchip_ATmega:ATmega32U4-M
- added U2: PRTR5V0U2X, Package_TO_SOT_SMD:SOT-143, symbol Power_Protection:PRTR5V0U2X
- added USB1: TYPE-C-31-M-12, Connector_USB:USB_C_Receptacle_HRO_TYPE-C-31-M-12, symbol Connector:USB_C_Receptacle_USB2.0
- J1: footprint Molex-0548190589:Reset_Pretty-Mask -> Connector_PinHeader_2.54mm:PinHeader_2x03_P2.54mm_Vertical; symbol cornelius-rescue:AVR-ISP-6-Connector -> Connector:AVR-ISP-6
- SW1: footprint locallib:SKQGADE010 -> Button_Switch_SMD:SW_SPST_SKQG_WithStem
- Y1: symbol cornelius-rescue:Crystal_GND24_Small-Device-Orbit-rescue-corne-plus-rescue -> Device:Crystal_GND24_Small
- renumbered D49 to ZD1
Connections:
- net +5V: now also U1.14 (VCC), U1.24 (AVCC), U1.34 (VCC), U1.44 (AVCC)
- net COL0: now also MX1.1, MX13.1, MX25.1, MX37.1, U1.41 (PF0)
- net COL1: now also MX14.1, MX2.1, MX26.1, MX38.1, U1.40 (PF1)
- net COL10: now also MX11.1, MX23.1, MX35.1, MX47.1, U1.27 (PD7)
- net COL11: now also MX12.1, MX24.1, MX36.1, MX48.1, U1.26 (PD6)
- net COL2: now also MX15.1, MX27.1, MX3.1, MX39.1, U1.39 (PF4)
- net COL3: now also MX16.1, MX28.1, MX4.1, MX40.1, U1.38 (PF5)
- net COL4: now also MX17.1, MX29.1, MX41.1, MX5.1, U1.37 (PF6)
- net COL5: now also MX18.1, MX30.1, MX42.1, MX6.1, U1.36 (PF7)
- net COL6: now also MX19.1, MX31.1, MX43.1, MX7.1, U1.31 (PC6)
- net COL7: now also MX20.1, MX32.1, MX44.1, MX8.1, U1.30 (PB6)
- net COL8: now also MX21.1, MX33.1, MX45.1, MX9.1, U1.29 (PB5)
- net COL9: now also MX10.1, MX22.1, MX34.1, MX46.1, U1.28 (PB4)
- net D+: now also R2.2, U2.2 (I/O1), USB1.A6 (D+), USB1.B6 (D+); no longer R2.1
- net D-: now also R3.2, U2.3 (I/O2), USB1.A7 (D-), USB1.B7 (D-); no longer R3.1
- net GND: now also U1.15 (GND), U1.23 (GND), U1.35 (GND), U1.43 (GND), U1.45 (GND), U1.5 (UGND), U2.1 (GND), USB1.A1 (GND), USB1.A12 (GND), USB1.B1 (GND), USB1.B12 (GND), USB1.S1 (SHIELD)
- net MISO: now also U1.11 (PB3)
- net MOSI: now also U1.10 (PB2)
- net RESET: now also U1.13 (~{RESET})
- net ROW0: now also U1.8 (PB0)
- net ROW1: now also U1.9 (PB1)
- net ROW3: now also U1.32 (PC7)
- net VBUS: now also U1.2 (UVCC), U1.7 (VBUS)
- net VCC: now also U2.4 (VCC), USB1.A4 (VBUS), USB1.A9 (VBUS), USB1.B4 (VBUS), USB1.B9 (VBUS)
- net at C2.1, Y1.3: now also U1.16 (XTAL2)
- net at C1.1, Y1.1: now also U1.17 (XTAL1)
- net at R1.2: now also U1.33 (~{HWB}/PE2)
- net at C3.1: now also U1.6 (UCAP)
- net at R4.1: now also USB1.B5 (CC2)
- net at R5.1: now also USB1.A5 (CC1)
- net at D1.2 (A): now also MX1.2
- net at D37.2 (A): now also MX37.2
- net at D38.2 (A): now also MX38.2
- net at D39.2 (A): now also MX39.2
- net at D7.2 (A): now also MX7.2
- net at D8.2 (A): now also MX8.2
- net at D9.2 (A): now also MX9.2
- net at D10.2 (A): now also MX10.2
- net at D11.2 (A): now also MX11.2
- net at D12.2 (A): now also MX12.2
- net at D19.2 (A): now also MX19.2
- net at D20.2 (A): now also MX20.2
- net at D21.2 (A): now also MX21.2
- net at D22.2 (A): now also MX22.2
- net at D23.2 (A): now also MX23.2
- net at D24.2 (A): now also MX24.2
- net at D31.2 (A): now also MX31.2
- net at D32.2 (A): now also MX32.2
- net at D33.2 (A): now also MX33.2
- net at D34.2 (A): now also MX34.2
- net at D35.2 (A): now also MX35.2
- net at D36.2 (A): now also MX36.2
- net at D46.2 (A): now also MX46.2
- net at D47.2 (A): now also MX47.2
- net at D48.2 (A): now also MX48.2
- net at D43.2 (A): now also MX43.2
- net at D44.2 (A): now also MX44.2
- net at D45.2 (A): now also MX45.2
- net at D2.2 (A): now also MX2.2
- net at D3.2 (A): now also MX3.2
- net at D4.2 (A): now also MX4.2
- net at D5.2 (A): now also MX5.2
- net at D6.2 (A): now also MX6.2
- net at D13.2 (A): now also MX13.2
- net at D14.2 (A): now also MX14.2
- net at D15.2 (A): now also MX15.2
- net at D16.2 (A): now also MX16.2
- net at D17.2 (A): now also MX17.2
- net at D18.2 (A): now also MX18.2
- net at D25.2 (A): now also MX25.2
- net at D26.2 (A): now also MX26.2
- net at D27.2 (A): now also MX27.2
- net at D28.2 (A): now also MX28.2
- net at D29.2 (A): now also MX29.2
- net at D30.2 (A): now also MX30.2
- net at D40.2 (A): now also MX40.2
- net at D41.2 (A): now also MX41.2
- net at D42.2 (A): now also MX42.2
- new net: R2.1, U1.4 (D+)
- new net: R3.1, U1.3 (D-)
Other:
- moved on the sheet: C3, D1, D10, D11, D12, D2, D3, D4, D5, D6, D7, D8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

Commit message: Add solder pcb
Parts:
- removed C1, C2: 22pF, Capacitor_SMD:C_0603_1608Metric, symbol Device:C_Small
- removed C3: 1uF, Capacitor_SMD:C_0603_1608Metric, symbol Device:C_Small
- removed C4, C5, C6: 0.1uF, Capacitor_SMD:C_0603_1608Metric, symbol Device:C_Small
- removed C7: 10uF, Capacitor_SMD:C_0603_1608Metric, symbol Device:C_Small
- removed D1, D10, D11, D12, D13, D14, D15, D16, D17, D18, D19, D2, D20, D21, D22, D23, D24, D25, D26, D27, D28, D29, D3, D30, D31, D32, D33, D34, D35, D36, D37, D38, D39, D4, D40, D41, D42, D43, D44, D45, D46, D47, D48, D5, D6, D7, D8, D9: SOD-123, Diode_SMD:D_SOD-123, symbol Device:D_Small
- removed F1: 500mA, Fuse:Fuse_1206_3216Metric, symbol Device:Polyfuse_Small
- removed J1: AVR-ISP-6, Connector_PinHeader_2.54mm:PinHeader_2x03_P2.54mm_Vertical, symbol Connector:AVR-ISP-6
- removed MX1, MX10, MX11, MX12, MX13, MX14, MX15, MX16, MX17, MX18, MX19, MX2, MX20, MX21, MX22, MX23, MX24, MX25, MX26, MX27, MX28, MX29, MX3, MX30, MX31, MX32, MX33, MX34, MX35, MX36, MX37, MX38, MX39, MX4, MX40, MX41, MX42, MX43, MX44, MX45, MX46, MX47, MX48, MX5, MX6, MX7, MX8, MX9: SW_Push, kbd:keyswitch_cherrymx_hotswap_1u, symbol Switch:SW_Push
- removed R1: 10k, Resistor_SMD:R_0805_2012Metric, symbol Device:R_Small
- removed R2, R3: 22, Resistor_SMD:R_0805_2012Metric, symbol Device:R_Small
- removed R4, R5: 5.1k, Resistor_SMD:R_0805_2012Metric, symbol Device:R_Small
- removed SW1: SW_Push, Button_Switch_SMD:SW_SPST_SKQG_WithStem, symbol Switch:SW_Push
- removed U1: ATmega32U4-M, Package_DFN_QFN:QFN-44-1EP_7x7mm_P0.5mm_EP5.2x5.2mm, symbol MCU_Microchip_ATmega:ATmega32U4-M
- removed U2: PRTR5V0U2X, Package_TO_SOT_SMD:SOT-143, symbol Power_Protection:PRTR5V0U2X
- removed USB1: TYPE-C-31-M-12, Connector_USB:USB_C_Receptacle_HRO_TYPE-C-31-M-12, symbol Connector:USB_C_Receptacle_USB2.0
- removed Y1: 16MHz, Crystal:Crystal_SMD_3225-4Pin_3.2x2.5mm, symbol Device:Crystal_GND24_Small
- removed ZD1: Schottky, Diode_SMD:D_SOD-123, symbol Device:D_Schottky_Small
Connections:
- no-connect marks 11 -> 0
Other:
- added sheet cornelius (../common/cornelius.kicad_sch)
- note removed: "ISP Header"
- note removed: "MCU"
- note removed: "PWR Flags"
- note removed: "Switch Matrix"
- note removed: "USB, ESD protection, Polyfuse"
