File: pcb/hotswap/cornelius.kicad_pcb (KiCad board)
At the start: 2 copper layers, 271.8 x 128.2 mm, 126 parts, among them J1 AVR-ISP-6, SW1 SW_Push, U1 ATmega32U4-MU, U2 PRTR5V0U2X, Y1 16MHz

Commit message: Add hotswap pcb
Parts:
- removed D49: Schottky, Diode_SMD:D_SOD-123
- added ZD1: Schottky, Diode_SMD:D_SOD-123, B.Cu at (144.4, 64.1)
- J1: footprint Molex-0548190589:Reset_Pretty-Mask -> Connector_PinHeader_2.54mm:PinHeader_2x03_P2.54mm_Vertical
- MX1, MX10, MX11, MX12, MX13, MX14, MX15, MX16, MX17, MX18, MX19, MX2, MX20, MX21, MX22, MX23, MX24, MX25, MX26, MX27, MX28, MX29, MX3, MX30, MX31, MX32, MX33, MX34, MX35, MX36, MX37, MX38, MX39, MX4, MX40, MX41, MX42, MX43, MX44, MX45, MX46, MX47, MX48, MX5, MX6, MX7, MX8, MX9: value MX-NoLED -> SW_Push; footprint MX_Only:MXOnly-1U-Hotswap -> kbd:keyswitch_cherrymx_hotswap_1u
- SW1: footprint locallib:SKQGADE010 -> Button_Switch_SMD:SW_SPST_SKQG_WithStem
- U1: value ATmega32U4-MU -> ATmega32U4-M; footprint Housings_DFN_QFN:QFN-44-1EP_7x7mm_Pitch0.5mm -> Package_DFN_QFN:QFN-44-1EP_7x7mm_P0.5mm_EP5.2x5.2mm
- U2: footprint locallib:SOT143B -> Package_TO_SOT_SMD:SOT-143
- USB1: value HRO-TYPE-C-31-M-12 -> TYPE-C-31-M-12; footprint Type-C:HRO-TYPE-C-31-M-12-Assembly -> Connector_USB:USB_C_Receptacle_HRO_TYPE-C-31-M-12
- moved USB1 3.65 mm to (148.5, 43.8)
- moved J1 2.95 mm to (156.5, 100.1)
- turned SW1 to 180 degrees
- turned U2 to 180 degrees
Connections:
- R2 pad 1: D+ -> Net-(U1-D+)
- R2 pad 2: Net-(R2-Pad2) -> D+
- R3 pad 1: D- -> Net-(U1-D-)
- R3 pad 2: Net-(R3-Pad2) -> D-
- R4 pad 1: Net-(R4-Pad1) -> Net-(USB1-CC2)
- R5 pad 1: Net-(R5-Pad1) -> Net-(USB1-CC1)
- U1 pad 1: Net-(U1-Pad1) -> unconnected-(U1-PE6-Pad1)
- U1 pad 12: Net-(U1-Pad12) -> unconnected-(U1-PB7-Pad12)
- U1 pad 18: Net-(U1-Pad18) -> unconnected-(U1-PD0-Pad18)
- U1 pad 19: Net-(U1-Pad19) -> unconnected-(U1-PD1-Pad19)
- U1 pad 20: Net-(U1-Pad20) -> unconnected-(U1-PD2-Pad20)
- U1 pad 21: Net-(U1-Pad21) -> unconnected-(U1-PD3-Pad21)
- U1 pad 22: Net-(U1-Pad22) -> unconnected-(U1-PD5-Pad22)
- U1 pad 25: Net-(U1-Pad25) -> unconnected-(U1-PD4-Pad25)
- U1 pad 3: D- -> Net-(U1-D-)
- U1 pad 4: D+ -> Net-(U1-D+)
- U1 pad 42: Net-(U1-Pad42) -> unconnected-(U1-AREF-Pad42)
- U2 pad 2: Net-(R2-Pad2) -> D+
- U2 pad 3: Net-(R3-Pad2) -> D-
Routing:
- net Net-(U1-D+): track 0.00 -> 55.1 mm
- net Net-(U1-D-): track 0.00 -> 55.1 mm
- net D-: track 55.1 -> 11.9 mm
- net D+: track 55.1 -> 12.4 mm
- net Net-(R2-Pad2): track 12.4 -> 0.00 mm
- net Net-(R3-Pad2): track 11.9 -> 0.00 mm
- net RESET: track 23.6 -> 30.0 mm
- net Net-(USB1-CC2): track 0.00 -> 6.36 mm, vias 0 -> 2
- net Net-(R4-Pad1): track 6.36 -> 0.00 mm, vias 2 -> 0
- net Net-(USB1-CC1): track 0.00 -> 6.30 mm, vias 0 -> 2
- net Net-(R5-Pad1): track 6.30 -> 0.00 mm, vias 2 -> 0
- net GND: track 202.9 -> 209.2 mm
Other:
- board text added: "CORNELIUS PCB Rev 1.1 202311"
- board text removed: "CORNELIUS PCB Rev 1.0 202101"

Commit message: Update jlcpcb files
Parts:
- MX1, MX10, MX11, MX12, MX13, MX14, MX15, MX16, MX17, MX18, MX19, MX2, MX20, MX21, MX22, MX23, MX24, MX25, MX26, MX27, MX28, MX29, MX3, MX30, MX31, MX32, MX33, MX34, MX35, MX36, MX37, MX38, MX39, MX4, MX40, MX41, MX42, MX43, MX44, MX45, MX46, MX47, MX48, MX5, MX6, MX7, MX8, MX9: moved to B.Cu
- turned MX1 to 170 degrees
- turned MX10 to -170 degrees
- turned MX11 to -170 degrees
- turned MX12 to -170 degrees
- turned MX13 to 170 degrees
- turned MX14 to 170 degrees
- turned MX15 to 170 degrees
- turned MX16 to 170 degrees
- turned MX17 to 170 degrees
- turned MX18 to 170 degrees
- turned MX19 to -170 degrees
- turned MX2 to 170 degrees
- turned MX20 to -170 degrees
- turned MX21 to -170 degrees
- turned MX22 to -170 degrees
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