File: pcb/solder/cornelius.kicad_pcb (KiCad board)
At the start: 2 copper layers, 271.8 x 128.2 mm, 126 parts, among them J1 AVR-ISP-6, SW1 SW_Push, U1 ATmega32U4-MU, U2 PRTR5V0U2X, Y1 16MHz

Commit message: Add solder pcb
Parts:
- removed D49: Schottky, Diode_SMD:D_SOD-123
- added ZD1: Schottky, Diode_SMD:D_SOD-123, B.Cu at (144.4, 64.1)
- J1: footprint Molex-0548190589:Reset_Pretty-Mask -> Connector_PinHeader_2.54mm:PinHeader_2x03_P2.54mm_Vertical
- MX1, MX10, MX11, MX12, MX13, MX14, MX15, MX16, MX17, MX18, MX19, MX2, MX20, MX21, MX22, MX23, MX24, MX25, MX26, MX27, MX28, MX29, MX3, MX30, MX31, MX32, MX33, MX34, MX35, MX36, MX37, MX38, MX39, MX4, MX40, MX41, MX42, MX43, MX44, MX45, MX46, MX47, MX48, MX5, MX6, MX7, MX8, MX9: value MX-NoLED -> SW_Push; footprint MX_Only:MXOnly-1U-NoLED -> kbd:keyswitch_cherrymx_hotswap_1u; moved to B.Cu
- SW1: footprint locallib:SKQGADE010 -> Button_Switch_SMD:SW_SPST_SKQG_WithStem
- U1: value ATmega32U4-MU -> ATmega32U4-M; footprint Housings_DFN_QFN:QFN-44-1EP_7x7mm_Pitch0.5mm -> Package_DFN_QFN:QFN-44-1EP_7x7mm_P0.5mm_EP5.2x5.2mm
- U2: footprint locallib:SOT143B -> Package_TO_SOT_SMD:SOT-143
- USB1: value HRO-TYPE-C-31-M-12 -> TYPE-C-31-M-12; footprint Type-C:HRO-TYPE-C-31-M-12-Assembly -> Connector_USB:USB_C_Receptacle_HRO_TYPE-C-31-M-12
- moved USB1 3.65 mm to (148.5, 43.8)
- moved J1 2.95 mm to (156.5, 100.1)
- turned MX1 to 170 degrees
- turned MX10 to -170 degrees
- turned MX11 to -170 degrees
- turned MX12 to -170 degrees
- turned MX13 to 170 degrees
- turned MX14 to 170 degrees
- turned MX15 to 170 degrees
- turned MX16 to 170 degrees
- turned MX17 to 170 degrees
- turned MX18 to 170 degrees
- turned MX19 to -170 degrees
- turned MX2 to 170 degrees
- turned MX20 to -170 degrees
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Connections:
- R2 pad 1: D+ -> Net-(U1-D+)
- R2 pad 2: Net-(R2-Pad2) -> D+
- R3 pad 1: D- -> Net-(U1-D-)
- R3 pad 2: Net-(R3-Pad2) -> D-
- R4 pad 1: Net-(R4-Pad1) -> Net-(USB1-CC2)
- R5 pad 1: Net-(R5-Pad1) -> Net-(USB1-CC1)
- U1 pad 1: Net-(U1-Pad1) -> unconnected-(U1-PE6-Pad1)
- U1 pad 12: Net-(U1-Pad12) -> unconnected-(U1-PB7-Pad12)
- U1 pad 18: Net-(U1-Pad18) -> unconnected-(U1-PD0-Pad18)
- U1 pad 19: Net-(U1-Pad19) -> unconnected-(U1-PD1-Pad19)
- U1 pad 20: Net-(U1-Pad20) -> unconnected-(U1-PD2-Pad20)
- U1 pad 21: Net-(U1-Pad21) -> unconnected-(U1-PD3-Pad21)
- U1 pad 22: Net-(U1-Pad22) -> unconnected-(U1-PD5-Pad22)
- U1 pad 25: Net-(U1-Pad25) -> unconnected-(U1-PD4-Pad25)
- U1 pad 3: D- -> Net-(U1-D-)
- U1 pad 4: D+ -> Net-(U1-D+)
- U1 pad 42: Net-(U1-Pad42) -> unconnected-(U1-AREF-Pad42)
- U2 pad 2: Net-(R2-Pad2) -> D+
- U2 pad 3: Net-(R3-Pad2) -> D-
Routing:
- net Net-(U1-D+): track 0.00 -> 55.1 mm
- net Net-(U1-D-): track 0.00 -> 55.1 mm
- net D-: track 55.1 -> 11.9 mm
- net D+: track 55.1 -> 12.4 mm
- net COL1: track 186.2 -> 172.0 mm, vias 1 -> 7
- net COL7: track 121.7 -> 109.3 mm, vias 1 -> 7
- net Net-(R2-Pad2): track 12.4 -> 0.00 mm
- net Net-(R3-Pad2): track 11.9 -> 0.00 mm
- net COL6: track 103.7 -> 92.1 mm, vias 1 -> 7
- net COL0: track 197.3 -> 185.8 mm, vias 1 -> 7
- net COL2: track 160.2 -> 149.2 mm, vias 1 -> 7
- net COL3: track 140.3 -> 129.4 mm, vias 1 -> 7
- net COL5: track 111.4 -> 100.5 mm, vias 1 -> 7
- net COL8: track 135.5 -> 124.6 mm, vias 1 -> 7
- net COL11: track 187.5 -> 176.7 mm, vias 1 -> 7
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Other:
- board text added: "CORNELIUS PCB Rev 1.1 202311"
- board text removed: "CORNELIUS Soldering PCB Rev 1.0 202101"

Commit message: Update solder pcb
Parts:
- MX1, MX10, MX11, MX12, MX13, MX14, MX15, MX16, MX17, MX18, MX19, MX2, MX20, MX21, MX22, MX23, MX24, MX25, MX26, MX27, MX28, MX29, MX3, MX30, MX31, MX32, MX33, MX34, MX35, MX36, MX37, MX38, MX39, MX4, MX40, MX41, MX42, MX43, MX44, MX45, MX46, MX47, MX48, MX5, MX6, MX7, MX8, MX9: footprint kbd:keyswitch_cherrymx_hotswap_1u -> kbd:keyswitch_cherrymx_alps_1u; moved to F.Cu
- turned MX1 to -10 degrees
- turned MX10 to 10 degrees
- turned MX11 to 10 degrees
- turned MX12 to 10 degrees
- turned MX13 to -10 degrees
- turned MX14 to -10 degrees
- turned MX15 to -10 degrees
- turned MX16 to -10 degrees
- turned MX17 to -10 degrees
- turned MX18 to -10 degrees
- turned MX19 to 10 degrees
- turned MX2 to -10 degrees
- turned MX20 to 10 degrees
- turned MX21 to 10 degrees
- turned MX22 to 10 degrees
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Routing:
- net GND: track 209.2 -> 171.5 mm
- net COL5: track 100.5 -> 109.0 mm, vias 7 -> 1
- net COL4: track 109.3 -> 117.6 mm, vias 7 -> 1
- net COL2: track 149.2 -> 157.2 mm, vias 7 -> 1
- net COL1: track 172.0 -> 179.8 mm, vias 7 -> 1
- net COL3: track 129.4 -> 137.2 mm, vias 7 -> 1
- net COL9: track 139.7 -> 146.7 mm, vias 7 -> 1
- net COL0: track 185.8 -> 192.8 mm, vias 7 -> 1
- net COL11: track 176.7 -> 183.5 mm, vias 7 -> 1
- net COL10: track 158.2 -> 164.9 mm, vias 7 -> 1
- net COL8: track 124.6 -> 128.7 mm, vias 7 -> 1
- net Net-(D19-A): track 4.80 -> 8.20 mm
- net Net-(D35-A): track 5.00 -> 8.40 mm
- net Net-(D31-A): track 4.84 -> 8.23 mm
- net Net-(D22-A): track 5.12 -> 8.50 mm
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