File: pcb/solder/cornelius.kicad_pcb (KiCad board)
At the start: 2 copper layers, 271.8 x 128.2 mm, 126 parts, among them J1 AVR-ISP-6, SW1 SW_Push, U1 ATmega32U4-M, U2 PRTR5V0U2X, Y1 16MHz

Commit message: Fix pass capacitor
Parts:
- moved ZD1 6.72 mm to (141.6, 58.0)
- moved C7 3.32 mm to (143.6, 112.4), turned to -90 degrees
Connections:
- F1 pad 1: VBUS -> +5V
- F1 pad 2: VCC -> VBUS
- U1 pad 2: VBUS -> +5V
- U1 pad 7: VBUS -> +5V
- U2 pad 4: VCC -> VBUS
- USB1 pad A4: VCC -> VBUS
- USB1 pad A9: VCC -> VBUS
- USB1 pad B4: VCC -> VBUS
- USB1 pad B9: VCC -> VBUS
- ZD1 pad 2: VBUS -> GND
Routing:
- net VBUS: track 61.4 -> 16.5 mm
- net +5V: track 109.4 -> 136.3 mm, vias 5 -> 7
- net VCC: track 16.5 -> 0.00 mm, vias 2 -> 0
- net GND: track 171.5 -> 174.0 mm, vias 4 -> 2
